File: open-bus-stop-pcb/open-bus-stop.kicad_sch (KiCad schematic)
At the start: 41 parts, among them J1 Conn_01x04_Pin, J2 Conn_01x02_Pin, J3 Conn_01x02, J5 Conn_01x02, P1 USB_C_Plug_USB2.0, SW2 SW_Push, SW4 SW_Push, U1 ESP32-C3-MINI-1, U2 DS3231M, U3 BQ24074RGT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

Commit message: (WIP) swapping RTCs and Display to decrease BOM cost
Parts:
- removed U2: DS3231M, Package_SO:SOIC-16W_7.5x10.3mm_P1.27mm, symbol Timer_RTC:DS3231M
- added C10: 3.3uF, symbol Device:C
- added C11, C12: 22pF, symbol Device:C
- added R13: 1k, symbol Device:R
- added U2: PCF8523T, Package_SO:SOIC-8_3.9x4.9mm_P1.27mm, symbol Timer_RTC:PCF8523T
- added Y1: 32.768kHz, symbol Device:Crystal
Connections:
- net GND: now also C10.1, C11.1, C12.1, U2.4 (VSS)
- net RTC_nIRQ: now also U2.7 (~{INT1}/CLKOUT)
- net SCL: now also U2.5 (SDA)
- net SDA: now also U2.6 (SCL)
- net VCC: now also R13.1
- net at BT1.1 (+): now also U2.3 (VBAT)
- net RTC_nRST: no longer names the net of U1.5 (GPIO2/ADC1_CH2)
- new net: C10.2, R13.2, U2.8 (VDD)
- new net: C12.2, U2.2 (OSCO), Y1.1
- new net: C11.2, U2.1 (OSCI), Y1.2
Other:
- moved on the sheet: BT1
